File: CH32V003_Breakout.kicad_pcb (KiCad board)
At the start: 2 copper layers, 13 parts, among them J1 PROG_HEADER, J2 USB_C, J3 HEADER_LEFT, J4 HEADER_RIGHT, SW1 NRST, U1 CH32V003FxUx, U2 AMS1117-2.85

Commit message: Started PCB Layout
Parts:
- U2: moved to F.Cu
- moved SW1 80.7 mm to (44.5, 38.1)
- moved J2 44.5 mm to (80.3, 27.2)
- moved R3 42.7 mm to (77.9, 33.3), turned to 180 degrees
- moved R2 40.5 mm to (82.7, 33.3)
- moved R1 24.7 mm to (65.7, 46.6), turned to 135 degrees
- moved J1 8.13 mm to (116.8, 77.5)
- moved C2 6.12 mm to (68.0, 64.4)
Connections:
- J4 pad 2: /PPBUS_3V3 -> /PPBUS_5V_USB
Routing:
- net GND: track 0.00 -> 4.84 mm, vias 0 -> 2
- net /PD4: track 0.00 -> 3.19 mm
- net /PD3: track 0.00 -> 3.15 mm
- net Net-(J2-CC2): track 0.00 -> 2.48 mm
- net Net-(J2-CC1): track 0.00 -> 2.47 mm
Other:
- board text added: "3.3V"
- board text added: "5V"
- board text added: "GND"
- board text added: "NRST|PD7"
- board text added: "OSCI|PA1"
- board text added: "OSCO|PA2"
- board text added: "PC0"
- board text added: "PC3"
- board text added: "PC4"
- board text added: "PC5|SCLK"
- board text added: "PC6|MOSI"
- board text added: "PC7|MISO"
- board text added: "PD0"
- board text added: "PD2|PU"
- board text added: "PD3|D-"
- board text added: "PD4|D+"
- board text added: "PD5|TX"
- board text added: "PD6|RX"
- board text added: "SCL|PC2"
- board text added: "SDA|PC1"
- board text added: "SWIO"

Commit message: V1.0 Board Release
Parts:
- J3, J4: moved to B.Cu
- SW1: footprint Button_Switch_SMD:SW_SPST_TL3342 -> Button_Switch_SMD:SW_SPST_CK_RS282G05A3
- U2: value AMS1117-2.85 -> AMS1117-3.3
- moved SW1 137.9 mm to (177.8, 73.4), turned to 0 degrees
- moved R1 119.1 mm to (183.7, 63.5), turned to -90 degrees
- moved C1 109.7 mm to (183.5, 53.0), turned to -90 degrees
- moved C2 105.3 mm to (173.3, 63.5), turned to 135 degrees
- moved R2 102.7 mm to (184.3, 48.0), turned to -90 degrees
- moved J2 99.2 mm to (177.8, 45.7)
- moved C3 99.0 mm to (172.1, 53.0), turned to 90 degrees
- moved R3 94.6 mm to (171.3, 48.0), turned to -90 degrees
- moved J1 58.5 mm to (175.3, 81.0)
- moved J3 55.8 mm to (168.9, 49.5), turned to 180 degrees
- moved U1 53.9 mm to (177.8, 64.8)
- moved J4 53.3 mm to (186.7, 49.5), turned to 180 degrees
- moved U2 30.9 mm to (177.8, 54.4), turned to 180 degrees
Routing:
- net /PPBUS_3V3: track 0.00 -> 54.5 mm, vias 0 -> 4
- net /NRST: track 0.00 -> 29.9 mm, vias 0 -> 2
- net /PD4: track 3.19 -> 26.8 mm, vias 0 -> 2
- net /PD3: track 3.15 -> 25.0 mm, vias 0 -> 2
- net /PD1: track 0.00 -> 17.7 mm, vias 0 -> 1
- net /PPBUS_5V_USB: track 0.00 -> 15.5 mm
- net /PC4: track 0.00 -> 13.2 mm
- net /PC5: track 0.00 -> 12.5 mm
- net /OSCI: track 0.00 -> 12.2 mm
- net /PD6: track 0.00 -> 12.1 mm
- net /PC3: track 0.00 -> 10.7 mm
- net /PD5: track 0.00 -> 10.6 mm
- net /MOSI: track 0.00 -> 10.5 mm
- net /OSCO: track 0.00 -> 10.4 mm
- net /PC0: track 0.00 -> 9.28 mm
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- added copper zone on F.Cu, net /PPBUS_3V3
- added copper zone on B.Cu, net GND
- added copper zone on F.Cu, net GND
Other:
- board outline added: 22 x 40 mm
- board text added: "CH32V003 Breakout Board"
- board text added: "RESET"
