File: CH32V003_Breakout.kicad_sch (KiCad schematic)
At the start: 13 parts, among them J1 PROG_HEADER, J2 USB_C, J3 HEADER_LEFT, J4 HEADER_RIGHT, SW1 NRST, U1 CH32V003FxUx, U2 AMS1117-2.85

Commit message: V1.0 Board Release
Parts:
- SW1: footprint Button_Switch_SMD:SW_SPST_TL3342 -> Button_Switch_SMD:SW_SPST_CK_RS282G05A3
- U2: value AMS1117-2.85 -> AMS1117-3.3; symbol Regulator_Linear:AMS1117-2.85 -> Regulator_Linear:AMS1117-3.3
Changed lines of the file:
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@@
 			)
 		)
-		(property "Footprint" "Button_Switch_SMD:SW_SPST_TL3342"
+		(property "Footprint" "Button_Switch_SMD:SW_SPST_CK_RS282G05A3"
 			(at 266.065 133.35 0)
 			(effects
@@
 	)
 	(symbol
-		(lib_id "Regulator_Linear:AMS1117-2.85")
+		(lib_id "Regulator_Linear:AMS1117-3.3")
 		(at 78.74 22.225 0)
 		(unit 1)
@@
 			)
 		)
-		(property "Value" "AMS1117-2.85"
+		(property "Value" "AMS1117-3.3"
 			(at 78.74 18.415 0)
 			(effects
@@
 			)
 		)
-		(property "Description" "1A Low Dropout regulator, positive, 2.85V fixed output, SOT-223"
+		(property "Description" "1A Low Dropout regulator, positive, 3.3V fixed output, SOT-223"
 			(at 78.74 22.225 0)
 			(effects
